File: Shift-out.sch (KiCad schematic (older format))
At the start: 23 parts, among them P1 CONN_02X08, P10 CONN_01X08, P11 CONN_01X02, P2 CONN_01X08, P3 CONN_02X08, P4 CONN_01X08, P5 INPUT, P6 CONN_02X08, P7 EXPANSION, P8 CONN_01X08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

Commit message: Modified output connector to allow direct servo plugging.
Parts:
- added P1, P13, P4, P8: CONN_01X08, Socket_Strips:Socket_Strip_Straight_1x08, symbol CONN_01X08
- renumbered P7 to P10, P8 to P11, P11 to P12, P9 to P14, P10 to P15, P1 to P2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
Connections:
- wire segments 201 -> 237
